File: kicad/low_cost_benchtop_ph_meter/low_cost_benchtop_ph_meter.kicad_pcb (KiCad board)
At the start: 2 copper layers, 50.8 x 22.9 mm, 10 parts, among them J1 Conn_01x16_Female, J2 Conn_01x12_Female, J3 Conn_Coaxial, U1 OPA128LM, U2 ADS1220xPW

Commit message: Week 6
Parts:
- added C1: 10 microF, Capacitor_SMD:C_0805_2012Metric, F.Cu at (144.2, 161.4)
- added C2: 10 microF, Capacitor_SMD:C_0805_2012Metric, F.Cu at (144.2, 164.4)
- added D1: LED, LED_SMD:LED_1206_3216Metric, F.Cu at (144.8, 158.2)
- added D2: BZV55B11, Diode_SMD:D_SOD-323, F.Cu at (148.6, 161.4)
- added D3: BAS316, Diode_SMD:D_SOD-323, F.Cu at (148.6, 164.3)
- added D4: BAS316, Diode_SMD:D_SOD-323, F.Cu at (148.6, 167.3)
- added R2: 5.6k, Resistor_SMD:R_0805_2012Metric, F.Cu at (144.2, 167.4)
- added R3: 9.1k, Resistor_SMD:R_1206_3216Metric, F.Cu at (150.5, 158.2)
- added R4: 1.01k, Resistor_SMD:R_0603_1608Metric, F.Cu at (152.7, 161.1)
- renumbered J1 to HatPins1, J2 to Hatpins2
Connections:
- net /GND renamed GND

Commit message: Week 8
Parts:
- added J1pHProbe1: Conn_Coaxial, BNCinp_31-5329:31532952RFX, F.Cu at (119.0, 150.6)
- added S1: DPDT Switch, center-off, B29AP_Switch:B29AP_NKK, F.Cu at (119.8, 160.3)
Connections:
- C1 pad 1: GND -> +9V
- C1 pad 2: unconnected-(C1-Pad2) -> GND
- C2 pad 1: unconnected-(C2-Pad1) -> GND
- C2 pad 2: GND -> -9V
- D1 pad 1: unconnected-(D1-K-Pad1) -> Net-(D1-K)
- D1 pad 2: unconnected-(D1-A-Pad2) -> Net-(D1-A)
- D2 pad 1: unconnected-(D2-K-Pad1) -> Net-(D1-K)
- D2 pad 2: unconnected-(D2-A-Pad2) -> Net-(D2-A)
- D3 pad 1: unconnected-(D3-K-Pad1) -> Net-(D3-K)
- D4 pad 2: unconnected-(D4-A-Pad2) -> Net-(D4-A)
- R2 pad 1: unconnected-(R2-Pad1) -> Net-(R2-Pad1)
- R2 pad 2: unconnected-(R2-Pad2) -> Net-(D2-A)
- R3 pad 1: unconnected-(R3-Pad1) -> Net-(U1-IN-)
- R3 pad 2: unconnected-(R3-Pad2) -> GND
- R4 pad 1: unconnected-(R4-Pad1) -> Net-(U1-OUTPUT)
- R4 pad 2: unconnected-(R4-Pad2) -> Net-(U1-IN-)
- U1 pad 1: unconnected-(U1-OFFSETTRIM-Pad1) -> Net-(R1-Pad1)
- U1 pad 2: unconnected-(U1-IN--Pad2) -> Net-(U1-IN-)
- U1 pad 3: unconnected-(U1-IN+-Pad3) -> Net-(J1pHProbe1-In)
- U1 pad 4: unconnected-(U1-VCC--Pad4) -> -9V
- U1 pad 5: unconnected-(U1-OFFSETTRIM-Pad5) -> Net-(R1-Pad3)
- U1 pad 6: unconnected-(U1-OUTPUT-Pad6) -> Net-(U1-OUTPUT)
- U1 pad 7: unconnected-(U1-VCC+-Pad7) -> +9V
- U1 pad 8: unconnected-(U1-SUBSTRATEANDCASE-Pad8) -> GND
